File: pir-light-hardware/pir-light-hardware.kicad_sch (KiCad schematic)
At the start: 44 parts, among them J1 ZH1.5-3, J2 ZH1.5-3, Q1 AON7240, Q2 NPN, Q3 PNP, Q4 PNP, U1 M74VHC1GT08DFT2G, U2 LMV331IDCKR, U3 AS312

Commit message: style: tweak schematic visuals
Parts:
- F1: value Fuse -> 300mA
Other:
- note added: "DIODE"
- note added: "RISKY"
Changed lines of the file:
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@@
 		)
 	)
+	(text "DIODE"
+		(exclude_from_sim no)
+		(at 184.785 121.92 0)
+		(effects
+			(font
+				(size 0.762 0.762)
+				(thickness 0.1524)
+				(bold yes)
+				(color 255 133 141 1)
+			)
+		)
+	)
 	(text "TO CHANGE"
 		(exclude_from_sim no)
@@
 		)
 	)
+	(text "RISKY"
+		(exclude_from_sim no)
+		(at 252.095 118.11 0)
+		(effects
+			(font
+				(size 0.762 0.762)
+				(thickness 0.1524)
+				(bold yes)
+				(color 255 133 141 1)
+			)
+		)
+	)
 	(text "TO CHANGE"
 		(exclude_from_sim no)
@@
 	(text "TO CHANGE"
 		(exclude_from_sim no)
+		(at 53.34 52.705 0)
+		(effects
+			(font
+				(size 0.762 0.762)
+				(thickness 0.1524)
+				(bold yes)
+				(color 255 133 141 1)
+			)
+		)
+	)
+	(text "TO CHANGE"
+		(exclude_from_sim no)
 		(at 200.025 114.935 0)
 		(effects
@@
 	(wire
 		(pts
-			(xy 189.865 122.555) (xy 188.595 122.555)
+			(xy 189.865 122.555) (xy 180.34 122.555)
 		)
 		(stroke
@@
 	)
 	(label "FB"
-		(at 188.595 122.555 180)
+		(at 180.34 122.555 180)
 		(effects
 			(font
@@
 		(dnp no)
 		(property "Reference" "Q4"
-			(at 201.295 108.585 0)
+			(at 200.025 107.95 90)
 			(show_name no)
 			(do_not_autoplace no)
@@
 		)
 		(property "Value" "PNP"
-			(at 198.755 108.585 0)
+			(at 200.025 110.49 90)
 			(show_name no)
 			(do_not_autoplace no)
@@
 		(in_pos_files yes)
 		(dnp no)
-		(fields_autoplaced yes)
 		(property "Reference" "F1"
-			(at 53.34 46.99 90)
+			(at 53.34 47.625 90)
 			(show_name no)
 			(do_not_autoplace no)
@@
 			)
 		)
-		(property "Value" "Fuse"
-			(at 53.34 49.53 90)
+		(property "Value" "300mA"
+			(at 53.34 50.165 90)
 			(show_name no)
 			(do_not_autoplace no)
