File: pir-light-hardware/pir-light-hardware.kicad_sch (KiCad schematic)
At the start: 44 parts, among them J1 ZH1.5-3, J2 ZH1.5-3, Q1 AON7240, Q2 NPN, Q3 PNP, Q4 PNP, U1 M74VHC1GT08DFT2G, U2 LMV331IDCKR, U3 AS312

Commit message: style: add notes to schematic
Other:
- note added: "1* If you plan to connect modules in a chain, populate this component only on the first and last device in the chain due to the resulting low equivalent parallel resistance."
- note added: "Note 1*"
- note added: "Note 2*"
- note removed: "RISKY"
Changed lines of the file:
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@@
 		(stroke
 			(width 0)
-			(type default)
+			(type dash_dot_dot)
+			(color 130 130 130 1)
 		)
 		(fill
@@
 	)
 	(rectangle
+		(start 249.301 114.3)
+		(end 257.556 120.65)
+		(stroke
+			(width 0)
+			(type dot)
+			(color 141 160 180 1)
+		)
+		(fill
+			(type none)
+		)
+	)
+	(rectangle
 		(start 30.48 39.37)
 		(end 267.335 134.62)
@@
 	)
 	(rectangle
+		(start 113.665 80.264)
+		(end 120.015 98.552)
+		(stroke
+			(width 0)
+			(type dot)
+			(color 141 160 180 1)
+		)
+		(fill
+			(type none)
+		)
+	)
+	(rectangle
 		(start 230.505 70.485)
 		(end 242.57 92.075)
@@
 	(text "DIODE"
 		(exclude_from_sim no)
-		(at 184.785 121.92 0)
-		(effects
-			(font
-				(size 0.762 0.762)
-				(thickness 0.1524)
-				(bold yes)
-				(color 255 133 141 1)
-			)
+		(at 184.658 122.682 0)
+		(effects
+			(font
+				(size 0.762 0.762)
+				(thickness 0.1524)
+				(bold yes)
+				(color 255 133 141 1)
+			)
+		)
+	)
+	(text "Note 2*"
+		(exclude_from_sim no)
+		(at 114.554 97.028 0)
+		(effects
+			(font
+				(size 0.762 0.762)
+				(thickness 0.1524)
+				(bold yes)
+				(color 145 194 119 1)
+			)
+			(justify left top)
 		)
 	)
@@
 		)
 	)
+	(text "1* If you plan to connect modules in a chain, populate this component only on the first and last device in the chain due to the resulting low equivalent parallel resistance.\n"
+		(exclude_from_sim no)
+		(at 47.625 144.145 0)
+		(effects
+			(font
+				(size 1.524 1.524)
+				(thickness 0.1524)
+				(bold yes)
+				(color 145 194 119 1)
+			)
+			(justify left top)
+		)
+	)
 	(text "TO CHANGE"
 		(exclude_from_sim no)
@@
 		)
 	)
-	(text "RISKY"
-		(exclude_from_sim no)
-		(at 252.095 118.11 0)
-		(effects
-			(font
-				(size 0.762 0.762)
-				(thickness 0.1524)
-				(bold yes)
-				(color 255 133 141 1)
-			)
-		)
-	)
+	(text "Note 1*"
+		(exclude_from_sim no)
+		(at 249.682 117.348 0)
+		(effects
+			(font
+				(size 0.762 0.762)
+				(thickness 0.1524)
+				(bold yes)
+				(color 145 194 119 1)
+			)
+			(justify left top)
+		)
+	)
