File: pir-light-hardware/pir-light-hardware.kicad_pcb (KiCad board)
At the start: 2 copper layers, 40 x 15 mm, 43 parts, among them J1 ZH1.5-3, J2 ZH1.5-3, Q1 DTA114EUAHE3-TP, Q2 AON7240, Q3 DTA114EUAHE3-TP, Q4 DTC114EUA-TP, U1 AS312, U2 M74VHC1GT08DFT2G, U3 LMV331IDCKR, U4 LMV331IDCKR

Commit message: style: add dimension values of pcb
Parts:
- moved C12 9.48 mm to (84.9, 114.2)
- moved C2 9.48 mm to (81.4, 111.4)
- moved C3 9.48 mm to (81.4, 113.3)
- moved C4 9.48 mm to (81.4, 115.3)
- moved C7 9.48 mm to (89.9, 112.6)
- moved F1 9.48 mm to (85.7, 125.4)
- moved JP1 9.48 mm to (77.7, 117.6)
- moved Q2 9.48 mm to (89.5, 117.0)
- moved R11 9.48 mm to (74.0, 109.5)
- moved R3 9.48 mm to (71.1, 109.5)
- moved R8 9.48 mm to (84.9, 119.2)
- moved C1 9.48 mm to (84.9, 111.6)
- moved C10 9.48 mm to (81.4, 125.2)
- moved C11 9.48 mm to (83.9, 107.5)
- moved C5 9.48 mm to (81.4, 117.3)
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